File: tp4056_kicad6_base/tp4056.kicad_pcb (KiCad board)
At the start: 2 copper layers, 41.8 x 20.5 mm, 21 parts, among them J1 USB_B_Micro, J2 Conn_01x01_Female, J3 Conn_01x01_Female, J4 Conn_01x01_Female, J5 Conn_01x01_Female, J6 Conn_01x01_Female, J7 Conn_01x01_Female, U1 TP4056, U2 DW01, U3 FS8205A

Commit message: update
Parts:
- R6: value ZERO -> 0R
Other:
- board text added: "1"
- board text added: "INGND"
- board text added: "INVCC"
- board text added: "OUTGND"
- board text added: "OUTVCC"
- board text added: "bat+"
- board text added: "bat-"
